Commit message: Optimize visual interaction and add voice interaction, etc.

File: src/ugv_main/ugv_description/urdf/bases/rasp_rover.xacro (robot description, xacro)
@@ -4,4 +4,7 @@
 <xacro:arg name="use_gazebo" default="false"/>
 <xacro:property name="use_gazebo" value="$(arg use_gazebo)"/>
+<xacro:macro name="GZ_VERSION" params="GZ_VERSION"></xacro:macro>
+<xacro:arg name="GZ_VERSION" default="classic"/>
+<xacro:property name="GZ_VERSION" value="$(arg GZ_VERSION)"/>
 <xacro:macro name="add_pt" params="add_pt"></xacro:macro>
 <xacro:arg name="add_pt" default="true"/>
@@ -20,7 +23,10 @@
 <xacro:if value="${add_pt}">
 <xacro:include filename="$(find ugv_description)/urdf/sensors/pt.xacro"/>
-<xacro:pt use_gazebo="$(arg use_gazebo)" pt_base_link_joint_pose_z="0.097648"/>
+<xacro:pt use_gazebo="$(arg use_gazebo)" GZ_VERSION="$(arg GZ_VERSION)" pt_base_link_joint_pose_z="0.097648" initial_positions_file="$(find ugv_description)/config/initial_positions.yaml"/>
 </xacro:if>
+<xacro:if value="${use_gazebo}">
 <xacro:include filename="$(find ugv_description)/urdf/gazebo/rasp_rover.gazebo"/>
+<xacro:gazebo GZ_VERSION="$(arg GZ_VERSION)"/>
+</xacro:if>
 <xacro:property name="base_inertial">
   <inertial>
@@ -58,78 +64,20 @@
   <xacro:insert_block name="base_joint_pose" />
 </joint>
-<xacro:property name="wheel_inertial_pose_z" value="0.027"/>
-<xacro:macro name="wheel_inertial" params="inertial_pose_z">
-  <inertial>
-    <origin xyz="0 0 ${inertial_pose_z}" rpy="0 0 0" />
-    <mass value="0.1153110" />
-    <inertia ixx="8.06312E-05" ixy="0" ixz="0" iyy="8.06312E-05" iyz="0" izz="0.000127361" />
-  </inertial>
-</xacro:macro>
-<xacro:property name="wheel_pose">
-  <origin xyz="0 0 0" rpy="1.5708 -0 0" />
-</xacro:property>
-<xacro:property name="up_wheel_joint_pose_x" value="0.0494657123506755"/>
-<xacro:property name="down_wheel_joint_pose_x" value="0.0475324306493252"/>
-<xacro:property name="wheel_joint_pose_y" value="0.0380100014305094"/>
-<xacro:property name="wheel_joint_pose_z" value="0.00674802802973084"/>
-<xacro:property name="wheel_joint_pose_rpy" value="-1.5708 0 0"/>
+<xacro:property name="up_wheel_joint_pose_x" value="0.049466"/>
+<xacro:property name="down_wheel_joint_pose_x" value="0.047532"/>
+<xacro:property name="wheel_joint_pose_y" value="0.06480"/>
+<xacro:property name="wheel_joint_pose_z" value="0.006748"/>
 <xacro:wheel wheel_prefix="left_up">
-  <xacro:wheel_inertial inertial_pose_z="${wheel_inertial_pose_z}"></xacro:wheel_inertial>
-  <xacro:insert_block name="wheel_pose" />
-  <origin xyz="${up_wheel_joint_pose_x} ${wheel_joint_pose_y} ${wheel_joint_pose_z}" rpy="${wheel_joint_pose_rpy}" />
+  <origin xyz="${up_wheel_joint_pose_x} ${wheel_joint_pose_y} ${wheel_joint_pose_z}" rpy="0 0 0" />
 </xacro:wheel>
 <xacro:wheel wheel_prefix="left_down">
-  <xacro:wheel_inertial inertial_pose_z="${wheel_inertial_pose_z}"></xacro:wheel_inertial>
-  <xacro:insert_block name="wheel_pose" />
-  <origin xyz="-${down_wheel_joint_pose_x} ${wheel_joint_pose_y} ${wheel_joint_pose_z}" rpy="${wheel_joint_pose_rpy}" />
+  <origin xyz="-${down_wheel_joint_pose_x} ${wheel_joint_pose_y} ${wheel_joint_pose_z}" rpy="0 0 0" />
 </xacro:wheel>
 <xacro:wheel wheel_prefix="right_up">
-  <xacro:wheel_inertial inertial_pose_z="-${wheel_inertial_pose_z}"></xacro:wheel_inertial>
-  <xacro:insert_block name="wheel_pose" />
-  <origin xyz="${up_wheel_joint_pose_x} -${wheel_joint_pose_y} ${wheel_joint_pose_z}" rpy="${wheel_joint_pose_rpy}" />
+  <origin xyz="${up_wheel_joint_pose_x} -${wheel_joint_pose_y} ${wheel_joint_pose_z}" rpy="0 0 0" />
 </xacro:wheel>
 <xacro:wheel wheel_prefix="right_down">
-  <xacro:wheel_inertial inertial_pose_z="-${wheel_inertial_pose_z}"></xacro:wheel_inertial>
-  <xacro:insert_block name="wheel_pose" />
-  <origin xyz="-${down_wheel_joint_pose_x} -${wheel_joint_pose_y} ${wheel_joint_pose_z}" rpy="${wheel_joint_pose_rpy}" />
+  <origin xyz="-${down_wheel_joint_pose_x} -${wheel_joint_pose_y} ${wheel_joint_pose_z}" rpy="0 0 0" />
 </xacro:wheel>
-<ros2_control name="WheelHardware" type="system">
-  <hardware>
-    <plugin>mock_components/GenericSystem</plugin>
-  </hardware>
-  <joint name="left_up_wheel_link_joint">
-    <command_interface name="position"/>
-    <state_interface name="position">
-      <param name="initial_value">0.0</param>
-    </state_interface>
-    <state_interface name="velocity">
-      <param name="initial_value">0.0</param>
-    </state_interface>
-  </joint>
-  <joint name="left_down_wheel_link_joint">
-    <command_interface name="position"/>
-    <state_interface name="position">
-      <param name="initial_value">0.0</param>
-    </state_interface>
-    <state_interface name="velocity">
-      <param name="initial_value">0.0</param>
-    </state_interface>
-  </joint>
-  <joint name="right_up_wheel_link_joint">
-    <command_interface name="position"/>
-    <state_interface name="position">
-      <param name="initial_value">0.0</param>
-    </state_interface>
-    <state_interface name="velocity">
-      <param name="initial_value">0.0</param>
-    </state_interface>
-  </joint>
-  <joint name="right_down_wheel_link_joint">
-    <command_interface name="position"/>
-    <state_interface name="position">
-      <param name="initial_value">0.0</param>
-    </state_interface>
-  </joint>
-</ros2_control>
 <xacro:include filename="$(arg urdf_extras)" />
 </robot>

File: src/ugv_main/ugv_description/urdf/bases/ugv_beast.xacro (robot description, xacro)
@@ -4,7 +4,13 @@
 <xacro:arg name="use_gazebo" default="false"/>
 <xacro:property name="use_gazebo" value="$(arg use_gazebo)"/>
+<xacro:macro name="GZ_VERSION" params="GZ_VERSION"></xacro:macro>
+<xacro:arg name="GZ_VERSION" default="classic"/>
+<xacro:property name="GZ_VERSION" value="$(arg GZ_VERSION)"/>
 <xacro:macro name="add_pt" params="add_pt"></xacro:macro>
 <xacro:arg name="add_pt" default="true"/>
 <xacro:property name="add_pt" value="$(arg add_pt)"/>
+<xacro:macro name="add_depth_camera" params="add_depth_camera"></xacro:macro>
+<xacro:arg name="add_depth_camera" default="false"/>
+<xacro:property name="add_depth_camera" value="$(arg add_depth_camera)"/>
 <xacro:arg name="robot_namespace" default="/" />
 <xacro:arg name="urdf_extras" default="empty.urdf" />
@@ -18,12 +24,17 @@
 <xacro:insert_block name="lidar_joint_pose" />
 </xacro:lidar>
+<xacro:unless value="${add_depth_camera}">
 <xacro:include filename="$(find ugv_description)/urdf/sensors/3d_camera.xacro" />
 <xacro:oak use_gazebo="$(arg use_gazebo)">
   <origin xyz="0.07031 0 0.0793" rpy="0 0 0" />
 </xacro:oak>
+</xacro:unless>
 <xacro:if value="${add_pt}">
 <xacro:include filename="$(find ugv_description)/urdf/sensors/pt.xacro"/>
-<xacro:pt use_gazebo="$(arg use_gazebo)" pt_base_link_joint_pose_z="0.0973"/>
+<xacro:pt use_gazebo="$(arg use_gazebo)"  GZ_VERSION="$(arg GZ_VERSION)" pt_base_link_joint_pose_z="0.0973" initial_positions_file="$(find ugv_description)/config/initial_positions.yaml"/>
+</xacro:if>
+<xacro:if value="${use_gazebo}">
 <xacro:include filename="$(find ugv_description)/urdf/gazebo/ugv_beast.gazebo"/>
+<xacro:gazebo GZ_VERSION="$(arg GZ_VERSION)"/>
 </xacro:if>
 <xacro:property name="base_inertial">
@@ -107,42 +118,4 @@
   <origin xyz="-${down_wheel_joint_pose_x} -${down_wheel_joint_pose_y} ${down_wheel_joint_pose_z}" rpy="${wheel_joint_pose_rpy}" />
 </xacro:wheel>
-<ros2_control name="WheelHardware" type="system">
-  <hardware>
-    <plugin>mock_components/GenericSystem</plugin>
-  </hardware>
-  <joint name="left_up_wheel_link_joint">
-    <command_interface name="position"/>
-    <state_interface name="position">
-      <param name="initial_value">0.0</param>
-    </state_interface>
-    <state_interface name="velocity">
-      <param name="initial_value">0.0</param>
-    </state_interface>
-  </joint>
-  <joint name="left_down_wheel_link_joint">
-    <command_interface name="position"/>
-    <state_interface name="position">
-      <param name="initial_value">0.0</param>
-    </state_interface>
-    <state_interface name="velocity">
-      <param name="initial_value">0.0</param>
-    </state_interface>
-  </joint>
-  <joint name="right_up_wheel_link_joint">
-    <command_interface name="position"/>
-    <state_interface name="position">
-      <param name="initial_value">0.0</param>
-    </state_interface>
-    <state_interface name="velocity">
-      <param name="initial_value">0.0</param>
-    </state_interface>
-  </joint>
-  <joint name="right_down_wheel_link_joint">
-    <command_interface name="position"/>
-    <state_interface name="position">
-      <param name="initial_value">0.0</param>
-    </state_interface>
-  </joint>
-</ros2_control>
 <xacro:include filename="$(arg urdf_extras)" />
 </robot>

File: src/ugv_main/ugv_description/urdf/bases/ugv_rover.xacro (robot description, xacro)
@@ -4,4 +4,7 @@
 <xacro:arg name="use_gazebo" default="false"/>
 <xacro:property name="use_gazebo" value="$(arg use_gazebo)"/>
+<xacro:macro name="GZ_VERSION" params="GZ_VERSION"></xacro:macro>
+<xacro:arg name="GZ_VERSION" default="classic"/>
+<xacro:property name="GZ_VERSION" value="$(arg GZ_VERSION)"/>
 <xacro:macro name="add_pt" params="add_pt"></xacro:macro>
 <xacro:arg name="add_pt" default="true"/>
@@ -29,12 +32,15 @@
 <xacro:if value="${add_pt}">
 <xacro:include filename="$(find ugv_description)/urdf/sensors/pt.xacro"/>
-<xacro:pt use_gazebo="$(arg use_gazebo)" pt_base_link_joint_pose_z="0.04"/>
+<xacro:pt use_gazebo="$(arg use_gazebo)" GZ_VERSION="$(arg GZ_VERSION)" pt_base_link_joint_pose_z="0.04" initial_positions_file="$(find ugv_description)/config/initial_positions.yaml"/>
+</xacro:if>
+<xacro:if value="${use_gazebo}">
 <xacro:include filename="$(find ugv_description)/urdf/gazebo/ugv_rover.gazebo"/>
+<xacro:gazebo GZ_VERSION="$(arg GZ_VERSION)"/>
 </xacro:if>
 <xacro:property name="base_inertial">
   <inertial>
-    <origin xyz="0.0 0 -0.018" rpy="0 0 0" />
-    <mass value="1.8601194" />
-    <inertia ixx="0.010769685" ixy="0" ixz="0" iyy="0.0118592" iyz="0" izz="0.017549519" />
+    <origin xyz="0.0 0 -0.0205" rpy="0 0 0" />
+    <mass value="2.1852443" />
+    <inertia ixx="0.012344031" ixy="0" ixz="0" iyy="0.01362398" iyz="0" izz="0.020616949" />
   </inertial>
 </xacro:property>
@@ -67,77 +73,19 @@
   <xacro:insert_block name="base_joint_pose" />
 </joint>
-<xacro:property name="wheel_inertial_pose_z" value="0.027"/>
-<xacro:macro name="wheel_inertial" params="inertial_pose_z">
-  <inertial>
-    <origin xyz="0 0 ${inertial_pose_z}" rpy="0 0 0" />
-    <mass value="0.1153110" />
-    <inertia ixx="8.06312E-05" ixy="0" ixz="0" iyy="8.06312E-05" iyz="0" izz="0.000127361" />
-  </inertial>
-</xacro:macro>
-<xacro:property name="wheel_pose">
-  <origin xyz="0 0 0" rpy="1.5708 -0 0" />
-</xacro:property>
 <xacro:property name="wheel_joint_pose_x" value="0.0855"/>
-<xacro:property name="wheel_joint_pose_y" value="0.06"/>
+<xacro:property name="wheel_joint_pose_y" value="0.08725"/>
 <xacro:property name="wheel_joint_pose_z" value="-0.041212"/>
-<xacro:property name="wheel_joint_pose_rpy" value="-1.5708 0 0"/>
 <xacro:wheel wheel_prefix="left_up">
-  <xacro:wheel_inertial inertial_pose_z="${wheel_inertial_pose_z}"></xacro:wheel_inertial>
-  <xacro:insert_block name="wheel_pose" />
-  <origin xyz="${wheel_joint_pose_x} ${wheel_joint_pose_y} ${wheel_joint_pose_z}" rpy="${wheel_joint_pose_rpy}" />
+  <origin xyz="${wheel_joint_pose_x} ${wheel_joint_pose_y} ${wheel_joint_pose_z}" rpy="0 0 0" />
 </xacro:wheel>
 <xacro:wheel wheel_prefix="left_down">
-  <xacro:wheel_inertial inertial_pose_z="${wheel_inertial_pose_z}"></xacro:wheel_inertial>
-  <xacro:insert_block name="wheel_pose" />
-  <origin xyz="-${wheel_joint_pose_x} ${wheel_joint_pose_y} ${wheel_joint_pose_z}" rpy="${wheel_joint_pose_rpy}" />
+  <origin xyz="-${wheel_joint_pose_x} ${wheel_joint_pose_y} ${wheel_joint_pose_z}" rpy="0 0 0" />
 </xacro:wheel>
 <xacro:wheel wheel_prefix="right_up">
-  <xacro:wheel_inertial inertial_pose_z="-${wheel_inertial_pose_z}"></xacro:wheel_inertial>
-  <xacro:insert_block name="wheel_pose" />
-  <origin xyz="${wheel_joint_pose_x} -${wheel_joint_pose_y} ${wheel_joint_pose_z}" rpy="${wheel_joint_pose_rpy}" />
+  <origin xyz="${wheel_joint_pose_x} -${wheel_joint_pose_y} ${wheel_joint_pose_z}" rpy="0 0 0" />
 </xacro:wheel>
 <xacro:wheel wheel_prefix="right_down">
-  <xacro:wheel_inertial inertial_pose_z="-${wheel_inertial_pose_z}"></xacro:wheel_inertial>
-  <xacro:insert_block name="wheel_pose" />
-  <origin xyz="-${wheel_joint_pose_x} -${wheel_joint_pose_y} ${wheel_joint_pose_z}" rpy="${wheel_joint_pose_rpy}" />
+  <origin xyz="-${wheel_joint_pose_x} -${wheel_joint_pose_y} ${wheel_joint_pose_z}" rpy="0 0 0" />
 </xacro:wheel>
-<ros2_control name="WheelHardware" type="system">
-  <hardware>
-    <plugin>mock_components/GenericSystem</plugin>
-  </hardware>
-  <joint name="left_up_wheel_link_joint">
-    <command_interface name="position"/>
-    <state_interface name="position">
-      <param name="initial_value">0.0</param>
-    </state_interface>
-    <state_interface name="velocity">
-      <param name="initial_value">0.0</param>
-    </state_interface>
-  </joint>
-  <joint name="left_down_wheel_link_joint">
-    <command_interface name="position"/>
-    <state_interface name="position">
-      <param name="initial_value">0.0</param>
-    </state_interface>
-    <state_interface name="velocity">
-      <param name="initial_value">0.0</param>
-    </state_interface>
-  </joint>
-  <joint name="right_up_wheel_link_joint">
-    <command_interface name="position"/>
-    <state_interface name="position">
-      <param name="initial_value">0.0</param>
-    </state_interface>
-    <state_interface name="velocity">
-      <param name="initial_value">0.0</param>
-    </state_interface>
-  </joint>
-  <joint name="right_down_wheel_link_joint">
-    <command_interface name="position"/>
-    <state_interface name="position">
-      <param name="initial_value">0.0</param>
-    </state_interface>
-  </joint>
-</ros2_control>
 <xacro:include filename="$(arg urdf_extras)" />
 </robot>

File: src/ugv_main/ugv_description/urdf/sensors/3d_camera.xacro (robot description, xacro)
@@ -38,4 +38,10 @@
 </xacro:if>
 <xacro:unless value="${use_gazebo}">
+<xacro:include filename="$(find depthai_descriptions)/urdf/include/depthai_macro.urdf.xacro" />
+<xacro:depthai_camera camera_name="oak" parent="3d_camera_link"
+  camera_model="OAK-D-LITE" base_frame="oak-d_frame"
+  cam_pos_x="0.017" cam_pos_y="0.0" cam_pos_z="0.005"
+  cam_roll="0.0" cam_pitch="0.0" cam_yaw="0.0"
+  rs_compat="false" />
 <link name="3d_camera_link">
   <inertial>

File: src/ugv_main/ugv_description/urdf/sensors/pt.xacro (robot description, xacro)
@@ -1,5 +1,6 @@
 <?xml version="1.0" ?>
 <robot name="pt" xmlns:xacro="http://www.ros.org/wiki/xacro">
-<xacro:macro name="pt" params="use_gazebo pt_base_link_joint_pose_z">
+<xacro:macro name="pt" params="use_gazebo GZ_VERSION pt_base_link_joint_pose_z initial_positions_file">
+<xacro:property name="initial_positions" value="${load_yaml(initial_positions_file)['initial_positions']}"/>
 <link name="pt_base_link">
   <inertial>
@@ -82,31 +83,4 @@
   </collision>
 </link>
-<xacro:if value="${use_gazebo}">
-<joint name="pt_base_link_joint" type="fixed">
-  <origin xyz="-0.02571 0 ${pt_base_link_joint_pose_z}" rpy="0 0 0" />
-  <parent link="base_link" />
-  <child link="pt_base_link" />
-  <axis xyz="0 0 0" />
-</joint>
-<joint name="pt_base_link_to_pt_link1" type="fixed">
-  <origin xyz="0.0113 0 0.0383" rpy="0 0 0" />
-  <parent link="pt_base_link" />
-  <child link="pt_link1" />
-  <axis xyz="0 0 0" />
-</joint>
-<joint name="pt_link1_to_pt_link2" type="fixed">
-  <origin xyz="0 0.02 0.043003" rpy="1.5708 0 0" />
-  <parent link="pt_link1" />
-  <child link="pt_link2" />
-  <axis xyz="0 0 0" />
-</joint>
-<joint name="pt_camera_link_joint" type="fixed">
-  <origin xyz="0.0484 -0.000569 0.02" rpy="-1.5708 0 0" />
-  <parent link="pt_link2" />
-  <child link="pt_camera_link" />
-  <axis xyz="0 0 0" />
-</joint>
-</xacro:if>
-<xacro:unless value="${use_gazebo}">
 <joint name="pt_base_link_joint" type="fixed">
   <origin xyz="-0.02571 0 ${pt_base_link_joint_pose_z}" rpy="0 0 0" />
@@ -120,5 +94,5 @@
   <child link="pt_link1" />
   <axis xyz="0 0 1" />
-  <limit lower="-3.14" upper="3.14" effort="0" velocity="0" />
+  <limit lower="-3.14" upper="3.14" effort="1.0" velocity="1.0" />
 </joint>
 <joint name="pt_link1_to_pt_link2" type="revolute">
@@ -127,5 +101,5 @@
   <child link="pt_link2" />
   <axis xyz="0 0 1" />
-  <limit lower="-0.5233333" upper="1.5707963" effort="0" velocity="0" />
+  <limit lower="-0.5233333" upper="1.5707963" effort="1.0" velocity="1.0" />
 </joint>
 <joint name="pt_camera_link_joint" type="fixed">
@@ -137,10 +111,22 @@
 <ros2_control name="PtHardware" type="system">
   <hardware>
+    <xacro:unless value="${use_gazebo}">
     <plugin>mock_components/GenericSystem</plugin>
+    </xacro:unless>
+    <xacro:if value="${use_gazebo}">
+      <xacro:if value="${GZ_VERSION == 'classic'}">
+        <plugin>gazebo_ros2_control/GazeboSystem</plugin>
+      </xacro:if>
+      <xacro:if value="${GZ_VERSION == 'harmonic'}">
+        <plugin>gz_ros2_control/GazeboSimSystem</plugin>
+      </xacro:if>
+    </xacro:if>
   </hardware>
   <joint name="pt_base_link_to_pt_link1">
     <command_interface name="position"/>
     <state_interface name="position">
-      <param name="initial_value">0.0</param>
+    <state_interface name="velocity"/>
+    <state_interface name="effort"/>
+      <param name="initial_value">${initial_positions['pt_base_link_to_pt_link1']}</param>
     </state_interface>
   </joint>
@@ -148,9 +134,40 @@
     <command_interface name="position"/>
     <state_interface name="position">
-      <param name="initial_value">0.0</param>
+    <state_interface name="velocity"/>
+    <state_interface name="effort"/>
+      <param name="initial_value">${initial_positions['pt_link1_to_pt_link2']}</param>
     </state_interface>
   </joint>
 </ros2_control>
-</xacro:unless>
- </xacro:macro>
+<transmission name="pt_base_link_to_pt_link1_transmission">
+  <type>transmission_interface/SimpleTransmission</type>
+  <joint name="pt_base_link_to_pt_link1">
+    <hardwareInterface>hardware_interface/EffortJointInterface</hardwareInterface>
+  </joint>
+  <actuator name="pt_base_link_to_pt_link1_actuator">
+    <mechanicalReduction>1</mechanicalReduction>
+  </actuator>
+</transmission>
+<transmission name="pt_link1_to_pt_link2_transmission">
+  <type>transmission_interface/SimpleTransmission</type>
+  <joint name="pt_link1_to_pt_link2">
+    <hardwareInterface>hardware_interface/EffortJointInterface</hardwareInterface>
+  </joint>
+  <actuator name="pt_link1_to_pt_link2_actuator">
+    <mechanicalReduction>1</mechanicalReduction>
+  </actuator>
+</transmission>
+<gazebo>
+  <xacro:if value="${GZ_VERSION == 'classic'}">
+    <plugin filename="libgazebo_ros2_control.so" name="gazebo_ros2_control">
+      <parameters>$(find ugv_description)/config/ros2_controllers.yaml</parameters>
+    </plugin>
+  </xacro:if>
+  <xacro:if value="${GZ_VERSION == 'harmonic'}">
+    <plugin name="gz_ros2_control::GazeboSimROS2ControlPlugin" filename="libgz_ros2_control-system.so">
+      <parameters>$(find ugv_description)/config/ros2_controllers.yaml</parameters>
+    </plugin>
+  </xacro:if>
+</gazebo>
+</xacro:macro>
 </robot>

File: src/ugv_main/ugv_description/urdf/wheels/rover_wheel.xacro (robot description, xacro)
@@ -1,18 +1,22 @@
 <?xml version="1.0" ?>
 <robot name="wheel" xmlns:xacro="http://www.ros.org/wiki/xacro">
-<xacro:macro name="wheel" params="wheel_prefix *inertial *link_pose *joint_pose">
+<xacro:macro name="wheel" params="wheel_prefix *joint_pose">
 <link name="${wheel_prefix}_wheel_link">
-  <xacro:insert_block name="inertial"/>
+  <inertial>
+    <origin xyz="0 0 0.0" rpy="0 0 0" />
+    <mass value="0.1625625" />
+    <inertia ixx="0.0000867" ixy="0" ixz="0" iyy="0.00013005" iyz="0" izz="0.0000867" />
+  </inertial>
   <visual>
-    <xacro:insert_block name="link_pose"/>
+    <origin xyz="0 0 0" rpy="0 0 0" />
     <geometry>
-      <mesh filename="file://$(find ugv_description)/meshes/wheels/rover/${wheel_prefix}_wheel_link.stl" />
+      <mesh filename="file://$(find ugv_description)/meshes/wheels/rover/wheel_link.stl" scale="1 1 1"/>
     </geometry>
     <material name="silver"/>
   </visual>
   <collision>
-    <xacro:insert_block name="link_pose"/>
+    <origin xyz="0 0 0" rpy="-1.5708 0 0"/>
     <geometry>
-      <mesh filename="file://$(find ugv_description)/meshes/wheels/rover/${wheel_prefix}_wheel_link.stl" />
+      <cylinder length="0.0425" radius="0.04" />
     </geometry>
   </collision>
@@ -22,5 +26,5 @@
   <parent link="base_link" />
   <child link="${wheel_prefix}_wheel_link" />
-  <axis xyz="0 0 1" />
+  <axis xyz="0 1 0" />
 </joint>
 </xacro:macro>
