Commit message: Organize and delete useless files

File: src/ugv_main/ugv_description/urdf/sensors/pt.xacro (robot description, xacro)
@@ -137,4 +137,37 @@
     <state_interface name="effort"/>
       <param name="initial_value">${initial_positions['pt_link1_to_pt_link2']}</param>
+    </state_interface>
+  </joint>
+  <joint name="left_up_wheel_link_joint">
+    <command_interface name="position"/>
+    <state_interface name="position">
+      <param name="initial_value">0.0</param>
+    </state_interface>
+    <state_interface name="velocity">
+      <param name="initial_value">0.0</param>
+    </state_interface>
+  </joint>
+  <joint name="left_down_wheel_link_joint">
+    <command_interface name="position"/>
+    <state_interface name="position">
+      <param name="initial_value">0.0</param>
+    </state_interface>
+    <state_interface name="velocity">
+      <param name="initial_value">0.0</param>
+    </state_interface>
+  </joint>
+  <joint name="right_up_wheel_link_joint">
+    <command_interface name="position"/>
+    <state_interface name="position">
+      <param name="initial_value">0.0</param>
+    </state_interface>
+    <state_interface name="velocity">
+      <param name="initial_value">0.0</param>
+    </state_interface>
+  </joint>
+  <joint name="right_down_wheel_link_joint">
+    <command_interface name="position"/>
+    <state_interface name="position">
+      <param name="initial_value">0.0</param>
     </state_interface>
   </joint>
